File: lm301h/lm301h_breakout.kicad_pcb (KiCad board)
At the start: 2 copper layers, 20.3 x 20.3 mm, 3 parts, among them J1 +, J2 -

Commit message: Add JLC PCB markings
Other:
- board text added: "JLCJLCJLCJLC"
Changed lines of the file:
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@@
+		)
+	)
+	(gr_text "JLCJLCJLCJLC"
+		(at 151.13 106.68 0)
+		(layer "B.SilkS")
+		(effects
+			(font
+				(size 0.9 0.9)
+				(thickness 0.1)
+			)
+			(justify mirror)
 		)
 	)
